Commit message: added gazebo control plugins and tags

File: urdf/brdlmillihexapod.urdf (robot description, URDF)
Before this commit: robot brdlmillihexapod_description, 19 links, 18 joints
Links:
- added link base_link
Joints:
- added joint j_brdlmillihexapod_attachment: type fixed, parent base_link, child torso, origin xyz=0 0 0 rpy=0 0 0
